File: pcb/inner.kicad_sch (KiCad schematic)
At the start: 4 parts, among them J10 FFC 10x1 0.5mm, J11 USB Breakout, J7 J7 Right Angle Connector, J8 J8 Mirror

Commit message: Revision 2
Parts:
- added J12: Activity LED Cathode, Connector_PinHeader_2.54mm:PinHeader_1x01_P2.54mm_Vertical, symbol Connector:Conn_01x01_Socket
Connections:
- net +3V: no longer J10.8 (Pin_8)
- new net ACT_LED_SINK: J10.8 (Pin_8), J12.1 (Pin_1)
Other:
- note added: "To implement an activity LED you want to bring out the - side, the cortex decides whether to sink this For 3.3V safety, use LED with voltage drop >= 1.7V"
